File: pcb/pcb.kicad_pcb (KiCad board)
At the start: 2 copper layers, 0 parts

Commit message: header in documentation fixed, pcb schematic done
Parts:
- added J1: Conn_02x04_Odd_Even, Connector_PinHeader_2.54mm:PinHeader_2x04_P2.54mm_Vertical, F.Cu at (101.6, 162.6)
- added J10: Conn_02x04_Odd_Even, Connector_PinHeader_2.54mm:PinHeader_2x04_P2.54mm_Vertical, F.Cu at (119.4, 121.9)
- added J11: Conn_02x04_Odd_Even, Connector_PinHeader_2.54mm:PinHeader_2x04_P2.54mm_Vertical, F.Cu at (137.2, 121.9)
- added J12: Conn_02x04_Odd_Even, Connector_PinHeader_2.54mm:PinHeader_2x04_P2.54mm_Vertical, F.Cu at (154.9, 121.9)
- added J13: Conn_02x04_Odd_Even, Connector_PinHeader_2.54mm:PinHeader_2x04_P2.54mm_Vertical, F.Cu at (101.6, 101.6)
- added J14: Conn_02x04_Odd_Even, Connector_PinHeader_2.54mm:PinHeader_2x04_P2.54mm_Vertical, F.Cu at (119.4, 101.6)
- added J15: Conn_02x04_Odd_Even, Connector_PinHeader_2.54mm:PinHeader_2x04_P2.54mm_Vertical, F.Cu at (137.2, 101.6)
- added J16: Conn_02x04_Odd_Even, Connector_PinHeader_2.54mm:PinHeader_2x04_P2.54mm_Vertical, F.Cu at (154.9, 101.6)
- added J17: Conn_02x04_Odd_Even, Connector_PinHeader_2.54mm:PinHeader_2x04_P2.54mm_Vertical, F.Cu at (101.6, 83.8)
- added J18: Conn_02x04_Odd_Even, Connector_PinHeader_2.54mm:PinHeader_2x04_P2.54mm_Vertical, F.Cu at (119.4, 83.8)
- added J19: Conn_02x04_Odd_Even, Connector_PinHeader_2.54mm:PinHeader_2x04_P2.54mm_Vertical, F.Cu at (137.2, 83.8)
- added J2: Conn_02x04_Odd_Even, Connector_PinHeader_2.54mm:PinHeader_2x04_P2.54mm_Vertical, F.Cu at (119.4, 162.6)
- added J20: Conn_02x04_Odd_Even, Connector_PinHeader_2.54mm:PinHeader_2x04_P2.54mm_Vertical, F.Cu at (154.9, 83.8)
- added J21: Conn_01x04_Pin, Connector_PinHeader_2.54mm:PinHeader_1x04_P2.54mm_Vertical, F.Cu at (152.4, 38.1)
- added J22: Conn_01x13_Pin, Connector_PinSocket_2.54mm:PinSocket_1x13_P2.54mm_Vertical, F.Cu at (116.8, 35.6)
- added J23: Conn_01x13_Pin, Connector_PinSocket_2.54mm:PinSocket_1x13_P2.54mm_Vertical, F.Cu at (132.1, 35.6)
- added J24: Conn_01x08_Pin, Connector_PinSocket_2.54mm:PinSocket_1x08_P2.54mm_Vertical, F.Cu at (162.6, 53.3)
- added J25: Conn_01x16_Pin, Connector_PinSocket_2.54mm:PinSocket_1x16_P2.54mm_Vertical, F.Cu at (177.8, 66.0)
- added J3: Conn_02x04_Odd_Even, Connector_PinHeader_2.54mm:PinHeader_2x04_P2.54mm_Vertical, F.Cu at (137.2, 162.6)
- added J4: Conn_02x04_Odd_Even, Connector_PinHeader_2.54mm:PinHeader_2x04_P2.54mm_Vertical, F.Cu at (154.9, 162.6)
- added J5: Conn_02x04_Odd_Even, Connector_PinHeader_2.54mm:PinHeader_2x04_P2.54mm_Vertical, F.Cu at (101.6, 142.2)
- added J6: Conn_02x04_Odd_Even, Connector_PinHeader_2.54mm:PinHeader_2x04_P2.54mm_Vertical, F.Cu at (119.4, 142.2)
- added J7: Conn_02x04_Odd_Even, Connector_PinHeader_2.54mm:PinHeader_2x04_P2.54mm_Vertical, F.Cu at (137.2, 142.2)
- added J8: Conn_02x04_Odd_Even, Connector_PinHeader_2.54mm:PinHeader_2x04_P2.54mm_Vertical, F.Cu at (154.9, 142.2)
- added J9: Conn_02x04_Odd_Even, Connector_PinHeader_2.54mm:PinHeader_2x04_P2.54mm_Vertical, F.Cu at (101.6, 121.9)
Routing:
- net Net-(J21-Pin_1): track 0.00 -> 69.6 mm
- net Net-(J21-Pin_2): track 0.00 -> 24.1 mm
- net Net-(J21-Pin_3): track 0.00 -> 17.3 mm
- net Net-(J21-Pin_4): track 0.00 -> 12.7 mm
Other:
- board text added: "A1"
- board text added: "CH0"
- board text added: "CH1"
- board text added: "CH10"
- board text added: "CH11"
- board text added: "CH12"
- board text added: "CH13"
- board text added: "CH14"
- board text added: "CH15"
- board text added: "CH2"
- board text added: "CH3"
- board text added: "CH4"
- board text added: "CH5"
- board text added: "CH6"
- board text added: "CH7"
- board text added: "CH8"
- board text added: "CH9"
- board text added: "D9"
- board text added: "RAW"
- board text added: "RST"
