File: pcb/pcb.kicad_sch (KiCad schematic)
At the start: 25 parts, among them J1 Conn_02x04_Odd_Even, J10 Conn_02x04_Odd_Even, J11 Conn_02x04_Odd_Even, J12 Conn_02x04_Odd_Even, J13 Conn_02x04_Odd_Even, J14 Conn_02x04_Odd_Even, J15 Conn_02x04_Odd_Even, J16 Conn_02x04_Odd_Even, J17 Conn_02x04_Odd_Even, J18 Conn_02x04_Odd_Even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

Commit message: rotated pcb, pcb documentation
Other:
- note added: "SCL"
- note added: "SDA"
- moved on the sheet: J1, J10, J11, J12, J13, J14, J15, J16, J17, J18, J19, J2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
